File: Racktemperatur.sch (KiCad schematic (older format))
At the start: 24 parts, among them J1 Conn_01x03, J2 Conn_01x03, J3 Barrel_Jack_MountingPin, J4 Screw_Terminal_01x02, Q1 IRLZ44N, U1 74HC595, U2 74HC595, U3 DS18B20, U4 L7805

Commit message: Minor changes
Other:
- moved on the sheet: R4
Changed lines of the file:
@@
 Wire Wire Line
 	4900 1050 4900 1200
-Wire Wire Line
-	6250 3500 3400 3500
 $Comp
 L Device:R R4
 U 1 1 5CAC6276
-P 3400 3650
-F 0 "R4" H 3470 3696 50  0000 L CNN
-F 1 "10kΩ" H 3470 3605 50  0000 L CNN
-F 2 "Resistor_SMD:R_0805_2012Metric_Pad1.15x1.40mm_HandSolder" V 3330 3650 50  0001 C CNN
-F 3 "~" H 3400 3650 50  0001 C CNN
-	1    3400 3650
-	1    0    0    -1
-$EndComp
-Wire Wire Line
-	3400 3500 3250 3500
-Wire Wire Line
-	3400 3800 3400 3950
+P 3400 3750
+F 0 "R4" H 3470 3796 50  0000 L CNN
+F 1 "10kΩ" H 3470 3705 50  0000 L CNN
+F 2 "Resistor_SMD:R_0805_2012Metric_Pad1.15x1.40mm_HandSolder" V 3330 3750 50  0001 C CNN
+F 3 "~" H 3400 3750 50  0001 C CNN
+	1    3400 3750
+	1    0    0    -1
+$EndComp
+Wire Wire Line
+	3400 3900 3400 3950
 Wire Wire Line
 	3400 3950 3800 3950
@@
 Wire Wire Line
 	3800 3950 3800 6350
-Connection ~ 3400 3500
 Wire Wire Line
 	2950 3300 2950 3200
@@
 NoConn ~ 9100 4950
 NoConn ~ 6450 5000
-NoConn ~ 8350 3700
 Wire Wire Line
 	5700 3200 5550 3200
@@
 Text Label 6350 1950 0    50   ~ 0
 5V
-Text Label 6350 2050 0    50   ~ 0
+Text Label 7200 2050 0    50   ~ 0
 3V3
 $Comp
@@
 Wire Wire Line
 	1300 3750 1400 3750
+Wire Wire Line
+	3250 3500 3400 3500
+Wire Wire Line
+	3400 3500 3400 3600
+Wire Wire Line
+	6250 3500 3400 3500
+Connection ~ 3400 3500
+NoConn ~ 1000 4150
 $EndSCHEMATC
