File: Racktemperatur.kicad_pcb (KiCad board)
At the start: 2 copper layers, 91.8 x 42.7 mm, 28 parts, among them J1 Conn_01x03, J2 Conn_01x03, J3 Barrel_Jack_MountingPin, J4 Screw_Terminal_01x02, Q1 IRLZ44N, U1 74HC595, U2 74HC595, U3 DS18B20, U4 L7805

Commit message: v1.7
Parts:
- removed the G*** at (111.7, 101.7) (x2)
- added G***: LOGO, haus-automatisierung:Logo2024-notext, F.Cu at (111.7, 101.7)
- added G***: LOGO, haus-automatisierung:Logo2024-notext, B.Cu at (111.7, 101.7)
Other:
- board text added: "v1.7"
- board text removed: "v1.6"
